File: PCB design/Motor_controller/Motor_controller.kicad_pcb (KiCad board)
At the start: 4 copper layers, 100.8 x 65 mm, 315 parts, among them J1 Conn_ARM_SWD_TagConnect_TC2030, J10 Conn_01x05_Pin, J11 532610371, J12 1984620, J13 1984617, J14 10067099-200LF, J15 Servo1, J16 Servo2, J17 Servo3, J18 Servo4, J19 Servo5, J2 SPI header, J20 Servo6, J3 I2C header, J4 UART header, J5 OLED header, J6 1984617, J7 USB4215-03-A, J8 B4B-XH-A, Q1 SL2302B, Q2 SL2302B, Q3 SL2302B, Q4 SL2302B, Q5 SI4447ADY-T1-GE3, U1 ATSAMD51N20A-AUT, U10 TLP3555ATP1_F, U11 NC7WZ14P6X, U12 TMC2208_SILENTSTEPSTICK, U13 DRV8311H, U14 DRV8231ADSG, U15 RIC11-31S10K2-GSMT, U2 FUSB302BMPX, U3 TPS2121RUXR, U4 LD1117S33TR_SOT223, U5 LM3489MMX_NOPB, U6 LM3489MMX_NOPB, U7 TLP3555ATP1_F, U8 TLP3555ATP1_F, U9 TLP3555ATP1_F, Y1 ECS-2333-160-BN-TR

Commit message: new file:   .gitignore 	new file:   .vscode/Motor_controller.mplab-local.json 	new file:   .vscode/Motor_controller.mplab.json 	new file:   .vscode/settings.json 	new file:   Firmware/Motor_controller.X/Motor_controller_default.bak0/components/FreeRTOS.yml 	new file:   Firmware/Motor_controller.X/Motor_controller_default.bak0/components/I2C/I2C.yml 	new file:   Firmware/Motor_controller.X/Motor_controller_default.bak0/components/I2C/components/sercom1.yml 	new file:   Firmware/Motor_controller.X/Motor_controller_default.bak0/components/O/O.yml 	new file:   Firmware/Motor_controller.X/Motor_controller_default.bak0/components/Sensor SPI/Sensor SPI.yml 	new file:   Firmware/Motor_controller.X/Motor_controller_default.bak0/components/Sensor SPI/components/sercom0.yml 	new file:   Firmware/Motor_controller.X/Motor_controller_default.bak0/components/Sensor SPU/Sensor SPU.yml 	new file:   Firmware/Motor_controller.X/Motor_controller_default.bak0/components/Ser/Ser.yml 	new file:   Firmware/Motor_controller.X/Motor_controller_default.bak0/components/Servo Motor/Servo Motor.yml 	new file:   Firmware/Motor_controller.X/Motor_controller_default.bak0/components/Servo Motor/components/sercom4.yml 	new file:   Firmware/Motor_controller.X/Motor_controller_default.bak0/components/UART/UART.yml 	new file:   Firmware/Motor_controller.X/Motor_controller_default.bak0/components/UART/components/sercom3.yml 	new file:   Firmware/Motor_controller.X/Motor_controller_default.bak0/components/UART/components/stdio.yml 	new file:   Firmware/Motor_controller.X/Motor_controller_default.bak0/components/cmsis.yml 	new file:   Firmware/Motor_controller.X/Motor_controller_default.bak0/components/core.yml 	new file:   Firmware/Motor_controller.X/Motor_controller_default.bak0/components/dfp.yml 	new file:   Firmware/Motor_controller.X/Motor_controller_default.bak0/components/eic.yml 	new file:   Firmware/Motor_controller.X/Motor_controller_default.bak0/components/evsys.yml 	new file:   Firmware/Motor_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
Parts:
- added R56: 1M, Resistor_SMD:R_1206_3216Metric, B.Cu at (72.4, 83.4)
- added R57: 1M, Resistor_SMD:R_1206_3216Metric, B.Cu at (111.0, 75.3)
- added R60: 1M, Resistor_SMD:R_1206_3216Metric, B.Cu at (80.8, 33.3)
- added R62: 1M, Resistor_SMD:R_1206_3216Metric, B.Cu at (112.6, 62.8)
Routing:
- net VBLDC: track 10.9 -> 17.1 mm
- net VServo: track 28.4 -> 32.1 mm
- net VSM: track 7.32 -> 9.39 mm
- net GND: track 228.7 -> 230.5 mm, vias 61 -> 62
- net VPM: track 14.8 -> 16.4 mm

Commit message: modified:   .vscode/Motor_controller.mplab.json 	new file:   Firmware/Doxyfile 	modified:   Firmware/Motor_controller.X/Motor_controller_default/components/FreeRTOS.yml 	modified:   Firmware/Motor_controller.X/Motor_controller_default/components/I2C/I2C.yml 	modified:   Firmware/Motor_controller.X/Motor_controller_default/components/I2C/components/sercom1.yml 	modified:   Firmware/Motor_controller.X/Motor_controller_default/components/Servo Motor/components/sercom4.yml 	deleted:    Firmware/Motor_controller.X/Motor_controller_default/components/X2Cscope.yml 	modified:   Firmware/Motor_controller.X/Motor_controller_default/components/adc0.yml 	modified:   Firmware/Motor_controller.X/Motor_controller_default/components/core.yml 	modified:   Firmware/Motor_controller.X/Motor_controller_default/components/evsys.yml 	modified:   Firmware/Motor_controller.X/Motor_controller_default/components/nvmctrl.yml 	modified:   Firmware/Motor_controller.X/Motor_controller_default/components/pmsm_foc.yml 	modified:   Firmware/Motor_controller.X/Motor_controller_default/components/pmsm_motor.yml 	modified:   Firmware/Motor_controller.X/Motor_controller_default/components/sercom3.yml 	modified:   Firmware/Motor_controller.X/Motor_controller_default/components/tcc0.yml 	modified:   Firmware/Motor_controller.X/Motor_controller_default/mcc-config.mc4 	modified:   Firmware/Motor_controller.X/mcc-manifest-autosave.yml 	modified:   Firmware/Motor_controller.X/mcc-manifest-generated-success.yml 	new file:   Firmware/src/BLDC/FOC_ADC.c 	new file:   Firmware/src/BLDC/FOC_ADC.h 	new file:   Firmware/src/BLDC/FOC_PWM.c 	new file:   Firmware/src/BLDC/FOC_PWM.h 	new file:   Firmware/src/BLDC/FOC_utilities.c 	new file:   Firmware/src/BLDC/FOC_utilities.h 	modified:   Firmware/src/config/default/QSpin/Field_Oriented_Control/mc_field_oriented_control.c 	modified:   Firmware/src/config/default/QSpin/Field_Oriented_Control/mc_field_oriented_control.h 	modified:   Firmware/src/config/default/QSpin/Field_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
Parts:
- moved kibuzzard-6A6AA48E 4.25 mm to (59.2, 46.8), turned to 180 degrees
- moved TP2 3.17 mm to (61.3, 46.8), turned to 90 degrees
- moved kibuzzard-6A6AA47F 2.53 mm to (59.2, 44.7), turned to 180 degrees
- moved TP7 0.43 mm to (61.3, 44.7), turned to 90 degrees
Connections:
- R39 pad 1: /SMDIR -> /SMDIR/PWMCL
- TP2 pad TP: /PWMCL -> /SMDIR/PWMCL
- U1 pad 41: /SMDIR -> /SMDIR/PWMCL
- U1 pad 42: /PWMCL -> /PWMBL
- U1 pad 43: /PWMBL -> /PWMAL
- U1 pad 44: /PWMAL -> unconnected-(U1-PC14-Pad44)
- U1 pad 45: /PWMAH -> /PWMCH
- U1 pad 47: /PWMCH -> /PWMAH
- U13 pad 20: /PWMCL -> /SMDIR/PWMCL
Routing:
- net /SMDIR/PWMCL: track 0.00 -> 79.3 mm, vias 0 -> 2
- net /SMDIR: track 54.2 -> 0.00 mm, vias 2 -> 0
- net /PWMCL: track 22.6 -> 0.00 mm, vias 1 -> 0
- net /PWMCH: track 24.9 -> 26.9 mm, vias 0 -> 2
- net /PWMAH: track 83.6 -> 85.6 mm, vias 3 -> 5

Commit message: Implemented FOC controller
Parts:
- removed kibuzzard-6A6AA47F: G***, kibuzzard-6A6AA47F
- removed kibuzzard-6A6AA48E: G***, kibuzzard-6A6AA48E
- added kibuzzard-6A9B0FE9: G***, kibuzzard-6A9B0FE9, F.Cu at (63.4, 44.7)
- added kibuzzard-6A9B0FFC: G***, kibuzzard-6A9B0FFC, F.Cu at (63.4, 46.8)
- R3: value 1k -> 200; moved to F.Cu
- R4, R5, R6, R7: value 200 -> 1k
- moved kibuzzard-6A6AB028 6.67 mm to (77.2, 53.5), turned to 90 degrees
- moved kibuzzard-6A6AB018 6.41 mm to (76.8, 46.7), turned to -90 degrees
- moved R3 6.25 mm to (78.2, 57.7), turned to 0 degrees
- moved C8 3.47 mm to (65.7, 52.1), turned to 90 degrees
- moved D4 3.25 mm to (99.3, 73.1)
- moved R39 3.22 mm to (95.9, 86.2)
- moved R40 2.85 mm to (95.9, 89.3)
- moved TP8 2.39 mm to (77.2, 51.3)
- moved R10 2.08 mm to (96.7, 75.4), turned to 0 degrees
- moved TP11 2.05 mm to (76.8, 48.9)
- moved C4 1.83 mm to (73.1, 52.5)
- moved Q3 1.81 mm to (96.8, 73.2), turned to 90 degrees
- moved R6 1.78 mm to (98.6, 70.9), turned to 0 degrees
- moved R36 0.25 mm to (104.6, 60.6)
Connections:
- R15 pad 1: /I2C_SCL -> /PD_SCL
- R16 pad 1: /I2C_SDA -> /PD_SDA
- R3 pad 1: Net-(U1-PC01) -> Net-(U1-PB05)
- R39 pad 1: /SMDIR/PWMCL -> /SMDIR
- TP2 pad TP: /SMDIR/PWMCL -> /PWMAH
- TP7 pad TP: /PWMCH -> /PWMAL
- U1 pad 10: unconnected-(U1-PB05-Pad10) -> Net-(U1-PB05)
- U1 pad 13: unconnected-(U1-PB06-Pad13) -> /PM_ADC
- U1 pad 14: /PMEN -> unconnected-(U1-PB07-Pad14)
- U1 pad 16: /SMEN -> unconnected-(U1-PB09-Pad16)
- U1 pad 26: /PM_ADC -> unconnected-(U1-PA08-Pad26)
- U1 pad 3: /PD_IRQ -> unconnected-(U1-PC00-Pad3)
- U1 pad 4: Net-(U1-PC01) -> unconnected-(U1-PC01-Pad4)
- U1 pad 40: /SMSTEP -> unconnected-(U1-PC10-Pad40)
- U1 pad 41: /SMDIR/PWMCL -> /PWMCL
- U1 pad 5: unconnected-(U1-PC02-Pad5) -> /SMDIR
- U1 pad 56: unconnected-(U1-PC16-Pad56) -> /UART_TX
- U1 pad 57: unconnected-(U1-PC17-Pad57) -> /UART_RX
- U1 pad 6: unconnected-(U1-PC03-Pad6) -> /SMEN
- U1 pad 61: unconnected-(U1-PC21-Pad61) -> /PD_IRQ
- U1 pad 7: /Servo_sel -> /PMEN
- U1 pad 72: /UART_RX -> /PD_SDA
- U1 pad 73: /UART_TX -> /PD_SCL
- U1 pad 99: unconnected-(U1-PB02-Pad99) -> /SMSTEP
- U13 pad 20: /SMDIR/PWMCL -> /PWMCL
- U2 pad 6: /I2C_SCL -> /PD_SCL
- U2 pad 7: /I2C_SDA -> /PD_SDA
Routing:
- net /SMDIR/PWMCL: track 79.3 -> 0.00 mm, vias 2 -> 0
- net /I2C_SDA: track 111.7 -> 72.1 mm, vias 2 -> 1
- net /SMDIR: track 0.00 -> 35.5 mm, vias 0 -> 1
- net /I2C_SCL: track 97.9 -> 67.9 mm
- net /PWMCL: track 0.00 -> 16.9 mm
- net /PD_SCL: track 0.00 -> 16.8 mm
- net /PD_SDA: track 0.00 -> 16.5 mm
- net /PD_IRQ: track 32.3 -> 19.5 mm
- net /SMEN: track 74.0 -> 62.7 mm, vias 4 -> 1
- net GND: track 230.5 -> 220.6 mm, vias 62 -> 60
- net Net-(D1-A): track 10.4 -> 1.51 mm, vias 1 -> 0
- net /SMSTEP: track 50.9 -> 42.0 mm, vias 2 -> 1
- net /PM_ADC: track 52.8 -> 45.7 mm, vias 2 -> 0
- net /PWMAL: track 80.2 -> 86.9 mm
- net +3.3V: track 503.3 -> 509.2 mm, vias 22 -> 20
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