File: PCB design/Motor_controller/Motor_controller.kicad_sch (KiCad schematic)
At the start: 77 parts, among them J1 Conn_ARM_SWD_TagConnect_TC2030, J2 SPI header, J3 I2C header, J4 UART header, J5 OLED header, Q1 SL2302B, Q2 SL2302B, Q3 SL2302B, Q4 SL2302B, U1 ATSAMD51N20A-AUT, Y1 ECS-2333-160-BN-TR

Commit message: modified:   .vscode/Motor_controller.mplab.json 	new file:   Firmware/Doxyfile 	modified:   Firmware/Motor_controller.X/Motor_controller_default/components/FreeRTOS.yml 	modified:   Firmware/Motor_controller.X/Motor_controller_default/components/I2C/I2C.yml 	modified:   Firmware/Motor_controller.X/Motor_controller_default/components/I2C/components/sercom1.yml 	modified:   Firmware/Motor_controller.X/Motor_controller_default/components/Servo Motor/components/sercom4.yml 	deleted:    Firmware/Motor_controller.X/Motor_controller_default/components/X2Cscope.yml 	modified:   Firmware/Motor_controller.X/Motor_controller_default/components/adc0.yml 	modified:   Firmware/Motor_controller.X/Motor_controller_default/components/core.yml 	modified:   Firmware/Motor_controller.X/Motor_controller_default/components/evsys.yml 	modified:   Firmware/Motor_controller.X/Motor_controller_default/components/nvmctrl.yml 	modified:   Firmware/Motor_controller.X/Motor_controller_default/components/pmsm_foc.yml 	modified:   Firmware/Motor_controller.X/Motor_controller_default/components/pmsm_motor.yml 	modified:   Firmware/Motor_controller.X/Motor_controller_default/components/sercom3.yml 	modified:   Firmware/Motor_controller.X/Motor_controller_default/components/tcc0.yml 	modified:   Firmware/Motor_controller.X/Motor_controller_default/mcc-config.mc4 	modified:   Firmware/Motor_controller.X/mcc-manifest-autosave.yml 	modified:   Firmware/Motor_controller.X/mcc-manifest-generated-success.yml 	new file:   Firmware/src/BLDC/FOC_ADC.c 	new file:   Firmware/src/BLDC/FOC_ADC.h 	new file:   Firmware/src/BLDC/FOC_PWM.c 	new file:   Firmware/src/BLDC/FOC_PWM.h 	new file:   Firmware/src/BLDC/FOC_utilities.c 	new file:   Firmware/src/BLDC/FOC_utilities.h 	modified:   Firmware/src/config/default/QSpin/Field_Oriented_Control/mc_field_oriented_control.c 	modified:   Firmware/src/config/default/QSpin/Field_Oriented_Control/mc_field_oriented_control.h 	modified:   Firmware/src/config/default/QSpin/Field_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
Connections:
- net SMDIR is gone; now on net SMDIR/PWMCL: U1.41 (PC11)
- net PWMAH: now also U1.47 (PA13); no longer U1.45 (PC15)
- net PWMAL: now also U1.43 (PC13); no longer U1.44 (PC14)
- net PWMBL: now also U1.42 (PC12); no longer U1.43 (PC13)
- net PWMCH: now also U1.45 (PC15); no longer U1.47 (PA13)
- net PWMCL renamed SMDIR/PWMCL
- net SMDIR/PWMCL: no longer U1.42 (PC12)
- no-connect marks 28 -> 29
Changed lines of the file:
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@@
 	)
 	(no_connect
+		(at 93.345 86.36)
+	)
+	(no_connect
 		(at 37.465 34.925)
 	)
@@
 	(wire
 		(pts
-			(xy 93.345 86.36) (xy 100.965 86.36)
-		)
-		(stroke
-			(width 0)
-			(type default)
-		)
-	)
-	(wire
-		(pts
 			(xy 17.78 41.275) (xy 17.78 42.545)
 		)
@@
 	(wire
 		(pts
-			(xy 133.35 153.67) (xy 140.97 153.67)
+			(xy 125.73 153.67) (xy 140.97 153.67)
 		)
 		(stroke
@@
 	(wire
 		(pts
+			(xy 93.345 81.28) (xy 100.584 81.28)
+		)
+		(stroke
+			(width 0)
+			(type default)
+		)
+	)
+	(wire
+		(pts
 			(xy 190.5 152.4) (xy 190.5 153.67)
 		)
@@
 	(wire
 		(pts
+			(xy 93.345 83.82) (xy 100.838 83.82)
+		)
+		(stroke
+			(width 0)
+			(type default)
+		)
+	)
+	(wire
+		(pts
 			(xy 93.345 76.2) (xy 101.6 76.2)
 		)
@@
 	(wire
 		(pts
+			(xy 29.845 60.325) (xy 37.465 60.325)
+		)
+		(stroke
+			(width 0)
+			(type default)
+		)
+	)
+	(wire
+		(pts
 			(xy 30.48 172.085) (xy 37.465 172.085)
 		)
@@
 	(wire
 		(pts
-			(xy 93.345 83.82) (xy 100.965 83.82)
-		)
-		(stroke
-			(width 0)
-			(type default)
-		)
-	)
-	(wire
-		(pts
 			(xy 184.785 156.21) (xy 202.565 156.21)
 		)
@@
 	(wire
 		(pts
-			(xy 93.345 78.74) (xy 101.6 78.74)
+			(xy 93.345 78.74) (xy 107.315 78.74)
 		)
 		(stroke
@@
 	(wire
 		(pts
-			(xy 93.345 81.28) (xy 100.965 81.28)
-		)
-		(stroke
-			(width 0)
-			(type default)
-		)
-	)
-	(wire
-		(pts
 			(xy 269.24 153.67) (xy 277.495 153.67)
 		)
@@
 	(wire
 		(pts
-			(xy 37.465 60.325) (xy 29.845 60.325)
-		)
-		(stroke
-			(width 0)
-			(type default)
-		)
-	)
-	(wire
-		(pts
 			(xy 257.175 126.365) (xy 275.59 126.365)
 		)
@@
 		)
 	)
-	(label "PWMCL"
-		(at 207.01 38.1 0)
-		(effects
-			(font
-				(size 1.27 1.27)
-			)
-			(justify left bottom)
-		)
-	)
 	(label "Servo2"
 		(at 29.21 70.485 0)
@@
 		)
 	)
+	(label "SMDIR{slash}PWMCL"
+		(at 125.73 153.67 0)
+		(effects
+			(font
+				(size 1.27 1.27)
+			)
+			(justify left bottom)
+		)
+	)
 	(label "SD_SCLK"
 		(at 28.575 80.645 0)
@@
 		)
 	)
-	(label "SMDIR"
-		(at 133.35 153.67 0)
-		(effects
-			(font
-				(size 1.27 1.27)
-			)
-			(justify left bottom)
-		)
-	)
 	(label "Servo_sel"
 		(at 27.94 32.385 0)
@@
 		)
 	)
-	(label "PWMCL"
-		(at 100.965 81.28 180)
-		(effects
-			(font
-				(size 1.27 1.27)
-			)
-			(justify right bottom)
-		)
-	)
 	(label "PDED_B"
 		(at 156.21 129.54 0)
@@
 		)
 	)
-	(label "SMDIR"
-		(at 101.6 78.74 180)
+	(label "PWMBL"
+		(at 100.584 81.28 180)
+		(effects
+			(font
+				(size 1.27 1.27)
+			)
+			(justify right bottom)
+		)
+	)
+	(label "SMDIR{slash}PWMCL"
+		(at 107.315 78.74 180)
 		(effects
 			(font
@@
 		)
 	)
-	(label "PWMCH"
-		(at 29.845 60.325 0)
-		(effects
-			(font
-				(size 1.27 1.27)
-			)
-			(justify left bottom)
-		)
-	)
 	(label "PWMBH"
 		(at 29.845 57.785 0)
@@
 		)
 	)
+	(label "PWMAH"
+		(at 29.845 60.325 0)
+		(effects
+			(font
+				(size 1.27 1.27)
+			)
+			(justify left bottom)
+		)
+	)
+	(label "SMDIR{slash}PWMCL"
+		(at 213.36 38.1 180)
+		(effects
+			(font
+				(size 1.27 1.27)
+			)
+			(justify right bottom)
+		)
+	)
 	(label "SMTX"
 		(at 133.35 158.115 0)
@@
 		)
 	)
-	(label "PWMAL"
-		(at 100.965 86.36 180)
-		(effects
-			(font
-				(size 1.27 1.27)
-			)
-			(justify right bottom)
-		)
-	)
 	(label "USB_DN"
 		(at 193.675 156.21 0)
@@
 		)
 	)
-	(label "PWMAH"
-		(at 100.965 88.9 180)
-		(effects
-			(font
-				(size 1.27 1.27)
-			)
-			(justify right bottom)
-		)
-	)
 	(label "SPI_SCK"
 		(at 29.21 40.005 0)
@@
 		)
 	)
-	(label "PWMBL"
-		(at 100.965 83.82 180)
+	(label "ServoEN"
+		(at 204.47 87.63 0)
 		(effects
 			(font
 				(size 1.27 1.27)
 			)
-			(justify right bottom)
+			(justify left bottom)
 		)
 	)
-	(label "ServoEN"
-		(at 204.47 87.63 0)
+	(label "I2C_SDA"
+		(at 267.335 126.365 0)
 		(effects
 			(font
@@
 		)
 	)
-	(label "I2C_SDA"
-		(at 267.335 126.365 0)
+	(label "PWMAL"
+		(at 100.838 83.82 180)
 		(effects
 			(font
 				(size 1.27 1.27)
 			)
-			(justify left bottom)
+			(justify right bottom)
 		)
 	)
@@
 		(effects
 			(font
+				(size 1.27 1.27)
+			)
+			(justify right bottom)
+		)
+	)
+	(label "PWMCH"
+		(at 100.965 88.9 180)
+		(effects
+			(font

Commit message: Implemented FOC controller
Parts:
- R3: value 1k -> 200
- R4, R5, R6, R7: value 200 -> 1k
Connections:
- net Servo_sel is gone; now on net PMEN: U1.7 (PA02)
- net PD_IRQ: now also U1.61 (PC21); no longer U1.3 (PC00)
- net PMEN: no longer U1.14 (PB07)
- net PM_ADC: now also U1.13 (PB06); no longer U1.26 (PA08)
- net PWMAH: now also TP2.TP
- net PWMAL: now also TP7.TP
- net PWMCH: no longer TP7.TP
- net SMEN: now also U1.6 (PC03); no longer U1.16 (PB09)
- net SMSTEP: now also U1.99 (PB02); no longer U1.40 (PC10)
- net UART_RX: now also U1.57 (PC17); no longer U1.72 (PA22)
- net UART_TX: now also U1.56 (PC16); no longer U1.73 (PA23)
- net at U1.10 (PB05): now also R3.1
- net at U1.4 (PC01): no longer R3.1
- net SMDIR: now reaches U1.5 (PC02)
- net SMDIR/PWMCL renamed PWMCL
- net PWMCL: no longer TP2.TP
- new net PD_SCL: U1.73 (PA23)
- new net PD_SDA: U1.72 (PA22)
- no-connect marks 29 -> 27
Other:
- note added: "ADC0_AIN10"
- note added: "ADC0_AIN11"
- note added: "ADC0_AIN9"
- note added: "SERCOM0_PAD0"
- note added: "SERCOM0_PAD1"
- note added: "SERCOM0_PAD2"
- note added: "SERCOM0_PAD3"
- note added: "SERCOM1_PAD0"
- note added: "SERCOM1_PAD1"
- note added: "SERCOM3_PAD0"
- note added: "SERCOM3_PAD1"
- note added: "SERCOM6_PAD0"
- note added: "SERCOM6_PAD1"
- note added: "TCC0_WO1"
- note added: "TCC0_WO2"
- note added: "TCC0_WO3"
- note added: "TCC0_WO5"
- note added: "TCC0_WO6"
- note added: "TCC0_WO7"
- moved on the sheet: D1, R3, TP2, TP7
