File: PCB design/Motor_controller/PM motor.kicad_sch (KiCad schematic)
At the start: 7 parts, among them J13 1984617, U14 DRV8231ADSG

Commit message: Implemented FOC controller
Other:
- note added: "2 Phase PM motor controller"
Changed lines of the file:
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@@
 	(generator_version "10.0")
 	(paper "A4")
+	(text "2 Phase PM motor controller"
+		(exclude_from_sim no)
+		(at 101.473 20.828 0)
+		(effects
+			(font
+				(size 7.62 7.62)
+				(thickness 1.524)
+				(bold yes)
+				(color 0 0 0 1)
+			)
+		)
+	)
 	(junction
 		(at 103.505 73.025)
