File: PCB design/Motor_controller/Power input.kicad_sch (KiCad schematic)
At the start: 27 parts, among them J6 1984617, J7 USB4215-03-A, Q5 SI4447ADY-T1-GE3, U2 FUSB302BMPX, U3 TPS2121RUXR

Commit message: Implemented FOC controller
Other:
- note added: "Power Input Bus & Power MUX"
- moved on the sheet: C10, C11, C12, C13, C14, C15, C16, C17, D6, D7, J6, J7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
