File: PCB design/Motor_controller/SD card.kicad_sch (KiCad schematic)
At the start: 9 parts, among them J14 10067099-200LF

Commit message: Implemented FOC controller
Other:
- note added: "SD Card Bus"
Changed lines of the file:
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@@
 	(generator_version "10.0")
 	(paper "A4")
+	(text "SD Card Bus"
+		(exclude_from_sim no)
+		(at 50.165 19.304 0)
+		(effects
+			(font
+				(size 7.62 7.62)
+				(thickness 1.524)
+				(bold yes)
+				(color 0 0 0 1)
+			)
+		)
+	)
 	(junction
 		(at 57.15 58.42)
