File: PCB design/Motor_controller/Servo_motor.kicad_sch (KiCad schematic)
At the start: 7 parts, among them J15 Servo1, J16 Servo2, J17 Servo3, J18 Servo4, J19 Servo5, J20 Servo6

Commit message: Implemented FOC controller
Other:
- note added: "Servo Motor Bus"
Changed lines of the file:
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@@
 	(generator_version "10.0")
 	(paper "A4")
+	(text "Servo Motor Bus"
+		(exclude_from_sim no)
+		(at 60.706 19.304 0)
+		(effects
+			(font
+				(size 7.62 7.62)
+				(thickness 1.524)
+				(bold yes)
+				(color 0 0 0 1)
+			)
+		)
+	)
 	(junction
 		(at 86.995 90.805)
