File: PCB design/Motor_controller/Stepper_motor.kicad_sch (KiCad schematic)
At the start: 22 parts, among them J10 Conn_01x05_Pin, J8 B4B-XH-A, U11 NC7WZ14P6X, U12 TMC2208_SILENTSTEPSTICK

Commit message: Implemented FOC controller
Other:
- note added: "Stepper Motor Driver"
Changed lines of the file:
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@@
 	(generator_version "10.0")
 	(paper "A4")
+	(text "Stepper Motor Driver"
+		(exclude_from_sim no)
+		(at 72.009 19.812 0)
+		(effects
+			(font
+				(size 7.62 7.62)
+				(thickness 1.524)
+				(bold yes)
+				(color 0 0 0 1)
+			)
+		)
+	)
 	(junction
 		(at 86.995 112.395)
